Commit message: Fix F/T sensor URDF

File: net_ft_description/urdf/net_ft_sensor.xacro (robot description, xacro)
@@ -46,5 +46,5 @@
     <link name="${prefix}fts_link">
       <visual>
-        <origin xyz="0 0 0" rpy="0 0 0" />
+        <origin xyz="0 0 ${sensor_height}" rpy="${pi} 0 0" />
         <geometry>
           <mesh filename="package://net_ft_description/meshes/visual/${mesh_file}.dae"/>
@@ -52,5 +52,5 @@
       </visual>
       <collision>
-        <origin xyz="0 0 0" rpy="0 0 0"/>
+        <origin xyz="0 0 ${sensor_height}" rpy="${pi} 0 0"/>
         <geometry>
           <mesh filename="package://net_ft_description/meshes/collision/${mesh_file}.stl"/>
