Commit message: Fix F/T sensor 3D model

File: net_ft_description/urdf/net_ft_sensor.urdf.xacro (robot description, xacro)
@@ -1,23 +1,23 @@
 <?xml version="1.0"?>
 <robot xmlns:xacro="http://wiki.ros.org/xacro" name="net_ft_sensor">
-    <!-- parameters -->
-    <xacro:arg name="ip_address" default="192.168.1.1" />
-    <xacro:arg name="rdt_sampling_rate" default="500" />
-    <xacro:arg name="sensor_type" default="ati_axia80" />
-    <xacro:arg name="bolts_mass" default="0.0" />
-    <xacro:arg name="internal_filter_rate" default="0" />
-    <xacro:arg name="use_hardware_biasing" default="false" />
-    <link name="world" />
-    <xacro:include filename="$(find net_ft_description)/urdf/net_ft_sensor.xacro" />
-    <xacro:net_ft_sensor
-      parent="world"
-      prefix=""
-      use_physical_hardware="false"
-      ip_address="$(arg ip_address)"
-      rdt_sampling_rate="$(arg rdt_sampling_rate)"
-      sensor_type="$(arg sensor_type)"
-      internal_filter_rate="$(arg internal_filter_rate)"
-      use_hardware_biasing="$(arg use_hardware_biasing)">
-        <origin xyz="0 0 0" rpy="0 0 0" />
-    </xacro:net_ft_sensor>
+  <!-- parameters -->
+  <xacro:arg name="ip_address" default="192.168.1.1" />
+  <xacro:arg name="rdt_sampling_rate" default="500" />
+  <xacro:arg name="sensor_type" default="ati_axia80" />
+  <xacro:arg name="bolts_mass" default="0.0" />
+  <xacro:arg name="internal_filter_rate" default="0" />
+  <xacro:arg name="use_hardware_biasing" default="false" />
+  <link name="world" />
+  <xacro:include filename="$(find net_ft_description)/urdf/net_ft_sensor.xacro" />
+  <xacro:net_ft_sensor
+    parent="world"
+    prefix=""
+    use_physical_hardware="false"
+    ip_address="$(arg ip_address)"
+    rdt_sampling_rate="$(arg rdt_sampling_rate)"
+    sensor_type="$(arg sensor_type)"
+    internal_filter_rate="$(arg internal_filter_rate)"
+    use_hardware_biasing="$(arg use_hardware_biasing)">
+    <origin xyz="0 0 0" rpy="0 0 0" />
+  </xacro:net_ft_sensor>
 </robot>

File: net_ft_description/urdf/net_ft_sensor.xacro (robot description, xacro)
@@ -16,44 +16,47 @@
         <mass value="${mass}" />
         <xacro:insert_block name="origin" />
-        <inertia ixx="${0.0833333 * mass * (3 * radius * radius + length * length)}" ixy="0.0" ixz="0.0"
-          iyy="${0.0833333 * mass * (3 * radius * radius + length * length)}" iyz="0.0"
+        <inertia ixx="${0.0833333 * mass * (3 * radius * radius + length * length)}"
+          ixy="0.0"
+          ixz="0.0"
+          iyy="${0.0833333 * mass * (3 * radius * radius + length * length)}"
+          iyz="0.0"
           izz="${0.5 * mass * radius * radius}" />
       </inertial>
     </xacro:macro>
     <xacro:if value="${sensor_type == 'ati_axia80'}">
-      <xacro:property name="mesh_file" value="ati_axia80_ft_sensor"/>
-      <xacro:property name="sensor_mass" value="0.28"/>
-      <xacro:property name="sensor_radius" value="0.082"/>
-      <xacro:property name="sensor_height" value="0.0254"/>
+      <xacro:property name="mesh_file" value="ati_axia80_ft_sensor" />
+      <xacro:property name="sensor_mass" value="0.28" />
+      <xacro:property name="sensor_radius" value="0.082" />
+      <xacro:property name="sensor_height" value="0.0254" />
     </xacro:if>
     <xacro:if value="${sensor_type == 'onrobot'}">
-      <xacro:property name="mesh_file" value="onrobot_hexe_v2_ft_sensor"/>
-      <xacro:property name="sensor_mass" value="0.245"/>
-      <xacro:property name="sensor_radius" value="0.07"/>
-      <xacro:property name="sensor_height" value="0.0375"/>
+      <xacro:property name="mesh_file" value="onrobot_hexe_v2_ft_sensor" />
+      <xacro:property name="sensor_mass" value="0.245" />
+      <xacro:property name="sensor_radius" value="0.07" />
+      <xacro:property name="sensor_height" value="0.0375" />
     </xacro:if>
     <xacro:if value="${sensor_type == 'ati'}">
-      <xacro:property name="mesh_file" value="ati_gamma_ip65_ft_sensor"/>
-      <xacro:property name="sensor_mass" value="0.5"/>
-      <xacro:property name="sensor_radius" value="0.07"/>
-      <xacro:property name="sensor_height" value="0.0375"/>
+      <xacro:property name="mesh_file" value="ati_gamma_ip65_ft_sensor" />
+      <xacro:property name="sensor_mass" value="0.5" />
+      <xacro:property name="sensor_radius" value="0.07" />
+      <xacro:property name="sensor_height" value="0.0375" />
     </xacro:if>
     <joint name="${prefix}fts_joint" type="fixed">
       <!-- The parent link must be read from the robot model it is attached to. -->
-      <parent link="${parent}"/>
-      <child link="${prefix}fts_link"/>
+      <parent link="${parent}" />
+      <child link="${prefix}fts_link" />
       <xacro:insert_block name="origin" />
     </joint>
     <link name="${prefix}fts_link">
       <visual>
-        <origin xyz="0 0 ${sensor_height}" rpy="${pi} 0 0" />
+        <origin xyz="0 0 0" rpy="0 0 0" />
         <geometry>
-          <mesh filename="package://net_ft_description/meshes/visual/${mesh_file}.dae"/>
+          <mesh filename="package://net_ft_description/meshes/visual/${mesh_file}.dae" />
         </geometry>
       </visual>
       <collision>
-        <origin xyz="0 0 ${sensor_height}" rpy="${pi} 0 0"/>
+        <origin xyz="0 0 0" rpy="0 0 0" />
         <geometry>
-          <mesh filename="package://net_ft_description/meshes/collision/${mesh_file}.stl"/>
+          <mesh filename="package://net_ft_description/meshes/collision/${mesh_file}.stl" />
         </geometry>
       </collision>
@@ -63,9 +66,9 @@
     </link>
     <joint name="${prefix}tool_side_joint" type="fixed">
-      <parent link="${prefix}fts_link"/>
-      <child link="${prefix}tool_mount_link"/>
-      <origin xyz="0 0 ${sensor_height}" rpy="0 0 0"/>
+      <parent link="${prefix}fts_link" />
+      <child link="${prefix}tool_mount_link" />
+      <origin xyz="0 0 ${sensor_height}" rpy="0 0 0" />
     </joint>
-    <link name="${prefix}tool_mount_link"/>
+    <link name="${prefix}tool_mount_link" />
     <xacro:if value="$(arg use_physical_hardware)">
       <xacro:include filename="$(find net_ft_description)/urdf/net_ft_sensor.ros2_control.xacro" />
@@ -76,5 +79,5 @@
         rdt_sampling_rate="${rdt_sampling_rate}"
         internal_filter_rate="${internal_filter_rate}"
-        use_hardware_biasing="${use_hardware_biasing}"/>
+        use_hardware_biasing="${use_hardware_biasing}" />
     </xacro:if>
   </xacro:macro>
